File: circuts/BH1772GLC.sch (KiCad schematic (older format))
At the start: 7 parts

Commit message: Pinout for BH1772GLC
Parts:
- removed C?: C, symbol C
- removed D?: LED, symbol LED
- removed Q?: 2N7002, symbol MOSFET_N
- removed R?: R1000, symbol R
- removed U?: IRU1015, symbol IRU1015
- removed U?: BH1772GLC, symbol BH1772GLC
- added C1: C, symbol C
- added D1: LED, symbol LED
- added K1: CONN_3, symbol CONN_3
- added Q1: 2N7002, symbol MOSFET_N
- added R2: R1000, symbol R
- added U1: BH1772GLC, symbol BH1772GLC
- gave numbers to parts that had none: 1
Connections:
- net +5V: now also C1.1, Q1.D, R2.1
- net GND: now also C1.2, U1.10 (GNDNC), U1.4 (GND_LED), U1.7 (GND)
- net at R1.1: now also D1.2 (K)
- new net: D1.1 (A), Q1.S
- new net: Q1.G, R2.2, U1.3 (LEDC)
- new net: K1.1 (P1), U1.5 (INT)
- new net: K1.2 (PM), U1.8 (SCL)
- new net: K1.3 (P3), U1.9 (SDA)
Changed lines of the file:
@@
-EESchema Schematic File Version 2  date Пн. 11 февр. 2013 23:52:02
+EESchema Schematic File Version 2  date Вт. 12 февр. 2013 22:38:41
 LIBS:power
 LIBS:device
@@
 LIBS:valves
 LIBS:asm
-EELAYER 43  0
+LIBS:BH1772GLC-cache
+EELAYER 25  0
 EELAYER END
 $Descr A4 11700 8267
@@
 Sheet 1 1
 Title ""
-Date "11 feb 2013"
+Date "12 feb 2013"
 Rev ""
 Comp ""
@@
 $EndDescr
 Wire Wire Line
+	6700 4200 6500 4200
+Wire Wire Line
+	6500 4200 6500 4350
+Wire Wire Line
+	6500 4350 6150 4350
+Wire Wire Line
+	6700 4000 6550 4000
+Wire Wire Line
+	6550 4000 6550 3850
+Wire Wire Line
+	6550 3850 6150 3850
+Wire Wire Line
+	4950 1750 4950 1900
+Wire Wire Line
 	5400 4750 5400 4950
 Wire Wire Line
@@
 	4750 3950 4450 3950
 Wire Wire Line
-	4900 3100 4900 2650
-Wire Wire Line
 	4600 3900 4600 3950
 Connection ~ 4600 3950
@@
 	4150 4700 4150 4800
 Wire Wire Line
-	4950 2750 4900 2750
-Connection ~ 4900 2750
-Wire Wire Line
 	5950 2750 6050 2750
 Wire Wire Line
@@
 	5600 4850 5200 4850
 Connection ~ 5400 4850
-$Comp
-L GND #PWR?
+Wire Wire Line
+	5200 1700 5200 1850
+Wire Wire Line
+	4900 3100 4900 2650
+Wire Wire Line
+	4900 2750 4950 2750
+Connection ~ 4900 2750
+Wire Wire Line
+	6700 4100 6350 4100
+Wire Wire Line
+	6350 4100 6350 4250
+Wire Wire Line
+	6350 4250 6150 4250
+$Comp
+L CONN_3 K1
+U 1 1 511A8C0E
+P 7050 4100
+F 0 "K1" V 7000 4100 50  0000 C CNN
+F 1 "CONN_3" V 7100 4100 40  0000 C CNN
+	1    7050 4100
+	1    0    0    -1
+$EndComp
+$Comp
+L +5V #PWR2
+U 1 1 511A7842
+P 4900 2650
+F 0 "#PWR2" H 4900 2740 20  0001 C CNN
+F 1 "+5V" H 4900 2740 30  0000 C CNN
+	1    4900 2650
+	1    0    0    -1
+$EndComp
+$Comp
+L PWR_FLAG #FLG1
+U 1 1 511A780B
+P 4950 1900
+F 0 "#FLG1" H 4950 1995 30  0001 C CNN
+F 1 "PWR_FLAG" H 4950 2080 30  0000 C CNN
+	1    4950 1900
+	-1   0    0    1
+$EndComp
+$Comp
+L PWR_FLAG #FLG2
+U 1 1 511A78AC
+P 5200 1700
+F 0 "#FLG2" H 5200 1795 30  0001 C CNN
+F 1 "PWR_FLAG" H 5200 1880 30  0000 C CNN
+	1    5200 1700
+	1    0    0    -1
+$EndComp
+$Comp
+L GND #PWR5
+U 1 1 511A77FC
+P 5200 1850
+F 0 "#PWR5" H 5200 1850 30  0001 C CNN
+F 1 "GND" H 5200 1780 30  0001 C CNN
+	1    5200 1850
+	1    0    0    -1
+$EndComp
+$Comp
+L +5V #PWR4
+U 1 1 511A77FA
+P 4950 1750
+F 0 "#PWR4" H 4950 1840 20  0001 C CNN
+F 1 "+5V" H 4950 1840 30  0000 C CNN
+	1    4950 1750
+	1    0    0    -1
+$EndComp
+$Comp
+L GND #PWR6
 U 1 1 51194B5A
 P 5400 4950
-F 0 "#PWR?" H 5400 4950 30  0001 C CNN
+F 0 "#PWR6" H 5400 4950 30  0001 C CNN
 F 1 "GND" H 5400 4880 30  0001 C CNN
 	1    5400 4950
@@
 3.3v
 $Comp
-L GND #PWR?
+L GND #PWR7
 U 1 1 511949EB
 P 5950 3050
-F 0 "#PWR?" H 5950 3050 30  0001 C CNN
+F 0 "#PWR7" H 5950 3050 30  0001 C CNN
 F 1 "GND" H 5950 2980 30  0001 C CNN
 	1    5950 3050
@@
 $EndComp
 $Comp
-L IRU1015 U?
-U 1 1 00000000
+L IRU1015 #U1
+U 1 1 511A77CF
 P 5450 2800
-F 0 "U?" H 5350 2750 60  0000 C CNN
+F 0 "#U1" H 5350 2750 60  0001 C CNN
 F 1 "IRU1015" H 5450 2950 60  0000 C CNN
 	1    5450 2800
@@
 $EndComp
 $Comp
-L GND #PWR?
+L GND #PWR1
 U 1 1 51193DBA
 P 4150 5450
-F 0 "#PWR?" H 4150 5450 30  0001 C CNN
+F 0 "#PWR1" H 4150 5450 30  0001 C CNN
 F 1 "GND" H 4150 5380 30  0001 C CNN
 	1    4150 5450
@@
 $EndComp
 $Comp
-L R R?
+L R R1
 U 1 1 51193DAE
 P 4150 5050
-F 0 "R?" V 4230 5050 50  0000 C CNN
+F 0 "R1" V 4230 5050 50  0000 C CNN
 F 1 "R68" V 4150 5050 50  0000 C CNN
 	1    4150 5050
@@
 $EndComp
 $Comp
-L LED D?
-U 1 1 00000000
+L LED D1
+U 1 1 511A77D0
 P 4150 4500
-F 0 "D?" H 4150 4600 50  0000 C CNN
+F 0 "D1" H 4150 4600 50  0000 C CNN
 F 1 "LED" H 4150 4400 50  0000 C CNN
 	1    4150 4500
@@
 $EndComp
 $Comp
-L +5V #PWR?
-U 1 1 00000000
-P 4900 2650
-F 0 "#PWR?" H 4900 2740 20  0001 C CNN
-F 1 "+5V" H 4900 2740 30  0000 C CNN
-	1    4900 2650
-	1    0    0    -1
-$EndComp
-$Comp
-L GND #PWR?
-U 1 1 00000000
+L GND #PWR3
+U 1 1 511A77D2
 P 4900 3600
-F 0 "#PWR?" H 4900 3600 30  0001 C CNN
+F 0 "#PWR3" H 4900 3600 30  0001 C CNN
 F 1 "GND" H 4900 3530 30  0001 C CNN
 	1    4900 3600
@@
 $EndComp
 $Comp
-L C C?
-U 1 1 00000000
+L C C1
+U 1 1 511A77D3
 P 4900 3300
-F 0 "C?" H 4950 3400 50  0000 L CNN
+F 0 "C1" H 4950 3400 50  0000 L CNN
 F 1 "C" H 4950 3200 50  0000 L CNN
 	1    4900 3300
@@
 $EndComp
 $Comp
-L R R?
-U 1 1 00000000
+L R R2
+U 1 1 511A77D4
 P 4600 3650
-F 0 "R?" V 4680 3650 50  0000 C CNN
+F 0 "R2" V 4680 3650 50  0000 C CNN
 F 1 "R1000" V 4600 3650 50  0000 C CNN
 	1    4600 3650
@@
 $EndComp
 $Comp
-L MOSFET_N Q?
-U 1 1 00000000
+L MOSFET_N Q1
+U 1 1 511A77D5
 P 4250 3950
-F 0 "Q?" H 4260 4120 60  0000 R CNN
+F 0 "Q1" H 4260 4120 60  0000 R CNN
 F 1 "2N7002" H 4300 3750 60  0000 R CNN
 	1    4250 3950
@@
 $EndComp
 $Comp
-L BH1772GLC U?
+L BH1772GLC U1
 U 1 1 00000000
 P 5450 4000
-F 0 "U?" H 5450 3800 60  0000 C CNN
-F 1 "BH1772GLC" H 5450 3900 60  0000 C CNN
+F 0 "U1" H 5400 3900 60  0000 C CNN
+F 1 "BH1772GLC" H 5550 4000 60  0000 C CNN
 	1    5450 4000
 	1    0    0    -1

Commit message: vanilla version.
Parts:
- removed K1: CONN_3, symbol CONN_3
- removed Q1: 2N7002, symbol MOSFET_N
- removed R1: R68, symbol R
- removed R2: R1000, symbol R
- added P1: CONN_4, symbol CONN_4
Connections:
- net +5V is gone; now on net +3.3V: C1.1
- net at D1.2 (K): now also U1.3 (LEDC)
- net +3.3V: now reaches D1.1 (A)
- net +3.3V: now also U1.6 (VCC), P1.1 (P1)
- net at U1.5 (INT): now also P1.2 (P2)
- net at U1.8 (SCL): now also P1.3 (P3)
- net at U1.9 (SDA): now also P1.4 (P4)
Other:
- moved on the sheet: D1
Changed lines of the file:
@@
-EESchema Schematic File Version 2  date Вт. 12 февр. 2013 22:38:41
+EESchema Schematic File Version 2  date Вс. 03 марта 2013 00:18:45
 LIBS:power
 LIBS:device
@@
 Sheet 1 1
 Title ""
-Date "12 feb 2013"
+Date "2 mar 2013"
 Rev ""
 Comp ""
@@
 $EndDescr
 Wire Wire Line
-	6700 4200 6500 4200
-Wire Wire Line
-	6500 4200 6500 4350
-Wire Wire Line
-	6500 4350 6150 4350
-Wire Wire Line
-	6700 4000 6550 4000
-Wire Wire Line
-	6550 4000 6550 3850
-Wire Wire Line
-	6550 3850 6150 3850
-Wire Wire Line
-	4950 1750 4950 1900
+	4600 3450 4600 3100
+Wire Wire Line
+	4600 3100 4900 3100
+Connection ~ 5200 4750
+Connection ~ 5200 4750
+Connection ~ 5400 4750
+Connection ~ 5600 4750
+Wire Wire Line
+	5450 3350 5450 3450
+Wire Wire Line
+	5600 2350 5600 2600
+Wire Wire Line
+	6700 3900 6700 3700
+Wire Wire Line
+	6150 4250 6350 4250
+Wire Wire Line
+	6350 4250 6350 4100
+Wire Wire Line
+	6350 4100 6700 4100
+Wire Wire Line
+	5850 2400 5850 2550
+Connection ~ 5400 4850
+Wire Wire Line
+	5600 4850 5200 4850
+Wire Wire Line
+	5600 4850 5600 4750
+Wire Wire Line
+	4900 3600 4900 3500
+Wire Wire Line
+	5200 4850 5200 4750
 Wire Wire Line
 	5400 4750 5400 4950
 Wire Wire Line
-	5200 4750 5200 4850
-Wire Wire Line
-	5950 2950 5950 3050
-Wire Wire Line
-	4150 5300 4150 5450
-Wire Wire Line
-	4150 4150 4150 4300
-Connection ~ 4600 3100
-Wire Wire Line
-	4150 3750 4150 3100
-Wire Wire Line
-	4150 3100 4900 3100
-Wire Wire Line
-	4600 3100 4600 3400
-Wire Wire Line
-	4900 3600 4900 3500
-Wire Wire Line
-	4750 3950 4450 3950
-Wire Wire Line
-	4600 3900 4600 3950
-Connection ~ 4600 3950
-Wire Wire Line
-	4150 4700 4150 4800
-Wire Wire Line
-	5950 2750 6050 2750
-Wire Wire Line
-	6050 2750 6050 3300
-Wire Wire Line
-	6050 3300 5450 3300
-Wire Wire Line
-	5450 3300 5450 3450
-Wire Wire Line
-	5600 4750 5600 4850
-Wire Wire Line
-	5600 4850 5200 4850
-Connection ~ 5400 4850
-Wire Wire Line
-	5200 1700 5200 1850
-Wire Wire Line
-	4900 3100 4900 2650
-Wire Wire Line
-	4900 2750 4950 2750
-Connection ~ 4900 2750
-Wire Wire Line
-	6700 4100 6350 4100
-Wire Wire Line
-	6350 4100 6350 4250
-Wire Wire Line
-	6350 4250 6150 4250
-$Comp
-L CONN_3 K1
-U 1 1 511A8C0E
-P 7050 4100
-F 0 "K1" V 7000 4100 50  0000 C CNN
-F 1 "CONN_3" V 7100 4100 40  0000 C CNN
-	1    7050 4100
-	1    0    0    -1
-$EndComp
-$Comp
-L +5V #PWR2
-U 1 1 511A7842
-P 4900 2650
-F 0 "#PWR2" H 4900 2740 20  0001 C CNN
-F 1 "+5V" H 4900 2740 30  0000 C CNN
-	1    4900 2650
-	1    0    0    -1
-$EndComp
-$Comp
-L PWR_FLAG #FLG1
+	6150 3850 6550 3850
+Wire Wire Line
+	6550 3850 6550 4000
+Wire Wire Line
+	6550 4000 6700 4000
+Wire Wire Line
+	6150 4350 6500 4350
+Wire Wire Line
+	6500 4350 6500 4200
+Wire Wire Line
+	6500 4200 6700 4200
+Wire Wire Line
+	4900 3100 4900 3000
+Wire Wire Line
+	4750 3950 4600 3950
+Wire Wire Line
+	4600 3950 4600 3850
+$Comp
+L +3.3V #PWR01
+U 1 1 513253D2
+P 5600 2350
+F 0 "#PWR01" H 5600 2310 30  0001 C CNN
+F 1 "+3.3V" H 5600 2460 30  0000 C CNN
+	1    5600 2350
+	1    0    0    -1
+$EndComp
+$Comp
+L +3.3V #PWR02
+U 1 1 513253B0
+P 4900 3000
+F 0 "#PWR02" H 4900 2960 30  0001 C CNN
+F 1 "+3.3V" H 4900 3110 30  0000 C CNN
+	1    4900 3000
+	1    0    0    -1
+$EndComp
+$Comp
+L +3.3V #PWR03
+U 1 1 513253A2
+P 5450 3350
+F 0 "#PWR03" H 5450 3310 30  0001 C CNN
+F 1 "+3.3V" H 5450 3460 30  0000 C CNN
+	1    5450 3350
+	1    0    0    -1
+$EndComp
+$Comp
+L +3.3V #PWR04
+U 1 1 5132540F
+P 6700 3700
+F 0 "#PWR04" H 6700 3660 30  0001 C CNN
+F 1 "+3.3V" H 6700 3810 30  0000 C CNN
+	1    6700 3700
+	1    0    0    -1
+$EndComp
+$Comp
+L CONN_4 P1
+U 1 1 00000000
+P 7050 4050
+F 0 "P1" V 7000 4050 50  0000 C CNN
+F 1 "CONN_4" V 7100 4050 50  0000 C CNN
+	1    7050 4050
+	1    0    0    -1
+$EndComp
+$Comp
+L PWR_FLAG #FLG05
 U 1 1 511A780B
-P 4950 1900
-F 0 "#FLG1" H 4950 1995 30  0001 C CNN
-F 1 "PWR_FLAG" H 4950 2080 30  0000 C CNN
-	1    4950 1900
+P 5600 2600
+F 0 "#FLG05" H 5600 2695 30  0001 C CNN
+F 1 "PWR_FLAG" H 5600 2780 30  0000 C CNN
+	1    5600 2600
 	-1   0    0    1
 $EndComp
 $Comp
-L PWR_FLAG #FLG2
+L PWR_FLAG #FLG06
 U 1 1 511A78AC
-P 5200 1700
-F 0 "#FLG2" H 5200 1795 30  0001 C CNN
-F 1 "PWR_FLAG" H 5200 1880 30  0000 C CNN
-	1    5200 1700
-	1    0    0    -1
-$EndComp
-$Comp
-L GND #PWR5
+P 5850 2400
+F 0 "#FLG06" H 5850 2495 30  0001 C CNN
+F 1 "PWR_FLAG" H 5850 2580 30  0000 C CNN
+	1    5850 2400
+	1    0    0    -1
+$EndComp
+$Comp
+L GND #PWR07
 U 1 1 511A77FC
-P 5200 1850
-F 0 "#PWR5" H 5200 1850 30  0001 C CNN
-F 1 "GND" H 5200 1780 30  0001 C CNN
-	1    5200 1850
-	1    0    0    -1
-$EndComp
-$Comp
-L +5V #PWR4
-U 1 1 511A77FA
-P 4950 1750
-F 0 "#PWR4" H 4950 1840 20  0001 C CNN
-F 1 "+5V" H 4950 1840 30  0000 C CNN
-	1    4950 1750
-	1    0    0    -1
-$EndComp
-$Comp
-L GND #PWR6
+P 5850 2550
+F 0 "#PWR07" H 5850 2550 30  0001 C CNN
+F 1 "GND" H 5850 2480 30  0001 C CNN
+	1    5850 2550
+	1    0    0    -1
+$EndComp
+$Comp
+L GND #PWR08
 U 1 1 51194B5A
 P 5400 4950
-F 0 "#PWR6" H 5400 4950 30  0001 C CNN
+F 0 "#PWR08" H 5400 4950 30  0001 C CNN
 F 1 "GND" H 5400 4880 30  0001 C CNN
 	1    5400 4950
 	1    0    0    -1
 $EndComp
-Text Label 5700 2850 0    60   ~ 0
-warning see datasheet!
-Text Label 5500 3450 0    60   ~ 0
-3.3v
-$Comp
-L GND #PWR7
-U 1 1 511949EB
-P 5950 3050
-F 0 "#PWR7" H 5950 3050 30  0001 C CNN
-F 1 "GND" H 5950 2980 30  0001 C CNN
-	1    5950 3050
-	1    0    0    -1
-$EndComp
-$Comp
-L IRU1015 #U1
-U 1 1 511A77CF
-P 5450 2800
-F 0 "#U1" H 5350 2750 60  0001 C CNN
-F 1 "IRU1015" H 5450 2950 60  0000 C CNN
-	1    5450 2800
-	1    0    0    -1
-$EndComp
-$Comp
-L GND #PWR1
-U 1 1 51193DBA
-P 4150 5450
-F 0 "#PWR1" H 4150 5450 30  0001 C CNN
-F 1 "GND" H 4150 5380 30  0001 C CNN
-	1    4150 5450
-	1    0    0    -1
-$EndComp
-$Comp
-L R R1
-U 1 1 51193DAE
-P 4150 5050
-F 0 "R1" V 4230 5050 50  0000 C CNN
-F 1 "R68" V 4150 5050 50  0000 C CNN
-	1    4150 5050
-	1    0    0    -1
-$EndComp
 $Comp
 L LED D1
 U 1 1 511A77D0
-P 4150 4500
-F 0 "D1" H 4150 4600 50  0000 C CNN
-F 1 "LED" H 4150 4400 50  0000 C CNN
-	1    4150 4500
+P 4600 3650
+F 0 "D1" H 4600 3750 50  0000 C CNN
+F 1 "LED" H 4600 3550 50  0000 C CNN
+	1    4600 3650
 	0    1    1    0
 $EndComp
 $Comp
-L GND #PWR3
+L GND #PWR010
 U 1 1 511A77D2
 P 4900 3600
-F 0 "#PWR3" H 4900 3600 30  0001 C CNN
+F 0 "#PWR010" H 4900 3600 30  0001 C CNN
 F 1 "GND" H 4900 3530 30  0001 C CNN
 	1    4900 3600
@@
 $EndComp
 $Comp
-L R R2
-U 1 1 511A77D4
-P 4600 3650
-F 0 "R2" V 4680 3650 50  0000 C CNN
-F 1 "R1000" V 4600 3650 50  0000 C CNN
-	1    4600 3650
-	1    0    0    -1
-$EndComp
-$Comp
-L MOSFET_N Q1
-U 1 1 511A77D5
-P 4250 3950
-F 0 "Q1" H 4260 4120 60  0000 R CNN
-F 1 "2N7002" H 4300 3750 60  0000 R CNN
-	1    4250 3950
-	-1   0    0    -1
-$EndComp
-$Comp
 L BH1772GLC U1
-U 1 1 00000000
+U 1 1 5132540E
 P 5450 4000
 F 0 "U1" H 5400 3900 60  0000 C CNN
