File: circuts/brain.sch (KiCad schematic (older format))
At the start: 23 parts, among them IC1 ATMEGA328P-A, K1 EKMS, P1 CONN_1, P2 CONN_1, P3 CONN_1, P4 UART, P5 I2C, P6 RGB, P7 CONN_1, P8 CONN_1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

Commit message: Bug fix (12v for LED)
Connections:
- net +12V: now also C2.1, C3.1, C4.1, P6.1 (P1)
- net GND: no longer C2.2, C3.2, C4.2, P6.1 (P1)
- net at P6.2 (P2), U1.17 (O2), U1.18 (O1): now also C2.2; no longer C2.1
- net at P6.3 (P3), U1.15 (O4), U1.16 (O3): now also C3.2; no longer C3.1
- net at P6.4 (P4), U1.13 (O6), U1.14 (O5): now also C4.2; no longer C4.1

Commit message: Fixed schematic (removed C for RGB)
Parts:
- removed C2, C3, C4: RGB, symbol CP1
Changed lines of the file:
@@
-EESchema Schematic File Version 2  date Сб. 23 февр. 2013 01:20:58
+EESchema Schematic File Version 2  date Вс. 24 февр. 2013 21:04:54
 LIBS:power
 LIBS:device
@@
 Sheet 1 1
 Title ""
-Date "22 feb 2013"
+Date "24 feb 2013"
 Rev ""
 Comp ""
@@
 $EndDescr
 Wire Wire Line
-	10150 3200 10150 3600
-Wire Wire Line
-	10150 3600 10300 3600
-Wire Wire Line
-	10300 3600 10300 3550
-Wire Wire Line
 	2700 3300 2700 3150
 Wire Wire Line
@@
 Wire Wire Line
 	8350 2700 6700 2700
-Connection ~ 10150 3400
 Wire Wire Line
 	10650 2800 10450 2800
@@
 	10200 2700 10650 2700
 Wire Wire Line
-	10400 3400 9900 3400
-Wire Wire Line
-	9900 3400 9900 3100
-Connection ~ 10150 2800
-Connection ~ 10400 3000
-Connection ~ 9900 2700
-Wire Wire Line
 	6700 2700 6700 2900
 Connection ~ 6700 2900
@@
 Wire Wire Line
 	10600 2500 10600 2450
-$Comp
-L +12V #PWR?
-U 1 1 5127E11D
-P 10300 3550
-F 0 "#PWR?" H 10300 3500 20  0001 C CNN
-F 1 "+12V" H 10300 3650 30  0000 C CNN
-	1    10300 3550
-	1    0    0    -1
-$EndComp
 $Comp
 L +12V #PWR?
@@
 $EndComp
 $Comp
-L CP1 C4
-U 1 1 5123A31D
-P 10400 3200
-F 0 "C4" H 10450 3300 50  0000 L CNN
-F 1 "RGB" H 10450 3100 50  0000 L CNN
-	1    10400 3200
-	-1   0    0    1
-$EndComp
-$Comp
-L CP1 C3
-U 1 1 5123A31B
-P 10150 3000
-F 0 "C3" H 10200 3100 50  0000 L CNN
-F 1 "RGB" H 10200 2900 50  0000 L CNN
-	1    10150 3000
-	-1   0    0    1
-$EndComp
-$Comp
-L CP1 C2
-U 1 1 5123A30D
-P 9900 2900
-F 0 "C2" H 9950 3000 50  0000 L CNN
-F 1 "RGB" H 9950 2800 50  0000 L CNN
-	1    9900 2900
-	-1   0    0    1
-$EndComp
-$Comp

Commit message: vanilla version.
Parts:
- removed U2: IRU1015, symbol IRU1015
- added U2: AP1117E33G, symbol AP1117E33G
Connections:
- net +12V: now also U2.3 (Vin)
- net +3.3V: now also U2.2 (Vout)
- net GND: now also U2.1 (Adj(GND))
Changed lines of the file:
@@
-EESchema Schematic File Version 2  date Вс. 24 февр. 2013 21:04:54
+EESchema Schematic File Version 2  date Сб. 02 марта 2013 21:32:09
 LIBS:power
 LIBS:device
@@
 encoding utf-8
 Sheet 1 1
-Title ""
-Date "24 feb 2013"
-Rev ""
+Title "Halligth v0.2"
+Date "2 mar 2013"
+Rev "2"
 Comp ""
 Comment1 ""
@@
 Comment4 ""
 $EndDescr
+$Comp
+L AP1117E33G U2
+U 1 1 51323685
+P 3300 2300
+F 0 "U2" H 3200 2250 60  0000 C CNN
+F 1 "AP1117E33G" H 3300 2450 60  0000 C CNN
+	1    3300 2300
+	1    0    0    -1
+$EndComp
 Wire Wire Line
 	2700 3300 2700 3150
@@
 	10600 2500 10600 2450
 $Comp
-L +12V #PWR?
+L +12V #PWR01
 U 1 1 5127E0C3
 P 10600 2450
-F 0 "#PWR?" H 10600 2400 20  0001 C CNN
+F 0 "#PWR01" H 10600 2400 20  0001 C CNN
 F 1 "+12V" H 10600 2550 30  0000 C CNN
 	1    10600 2450
@@
 $EndComp
 $Comp
-L IRU1015 U2
-U 1 1 5123DEC5
-P 3300 2300
-F 0 "U2" H 3200 2250 60  0000 C CNN
-F 1 "IRU1015" H 3300 2450 60  0000 C CNN
-	1    3300 2300
-	1    0    0    -1
-$EndComp
-$Comp
-L GND #PWR01
+L GND #PWR02
 U 1 1 5123DDB1
 P 2700 3300
-F 0 "#PWR01" H 2700 3300 30  0001 C CNN
+F 0 "#PWR02" H 2700 3300 30  0001 C CNN
 F 1 "GND" H 2700 3230 30  0001 C CNN
 	1    2700 3300
@@
 $EndComp
 $Comp
-L +12V #PWR02
+L +12V #PWR03
 U 1 1 5123DDAE
 P 2700 2800
-F 0 "#PWR02" H 2700 2750 20  0001 C CNN
+F 0 "#PWR03" H 2700 2750 20  0001 C CNN
 F 1 "+12V" H 2700 2900 30  0000 C CNN
 	1    2700 2800
@@
 $EndComp
 $Comp
-L +3,3V #PWR03
+L +3,3V #PWR04
 U 1 1 5123BC81
 P 7250 5450
-F 0 "#PWR03" H 7250 5410 30  0001 C CNN
+F 0 "#PWR04" H 7250 5410 30  0001 C CNN
 F 1 "+3,3V" H 7250 5560 30  0000 C CNN
 	1    7250 5450
@@
 NoConn ~ 4600 3200
 $Comp
-L PWR_FLAG #FLG04
+L PWR_FLAG #FLG05
 U 1 1 5123A541
 P 5050 1550
-F 0 "#FLG04" H 5050 1645 30  0001 C CNN
+F 0 "#FLG05" H 5050 1645 30  0001 C CNN
 F 1 "PWR_FLAG" H 5050 1730 30  0000 C CNN
 	1    5050 1550
@@
 $EndComp
 $Comp
-L PWR_FLAG #FLG05
+L PWR_FLAG #FLG06
 U 1 1 5123A550
 P 5350 1400
-F 0 "#FLG05" H 5350 1495 30  0001 C CNN
+F 0 "#FLG06" H 5350 1495 30  0001 C CNN
 F 1 "PWR_FLAG" H 5350 1580 30  0000 C CNN
 	1    5350 1400
@@
 $EndComp
 $Comp
-L GND #PWR06
+L GND #PWR07
 U 1 1 5123A527
 P 5350 1550
-F 0 "#PWR06" H 5350 1550 30  0001 C CNN
+F 0 "#PWR07" H 5350 1550 30  0001 C CNN
 F 1 "GND" H 5350 1480 30  0001 C CNN
 	1    5350 1550
@@
 $EndComp
 $Comp
-L +12V #PWR07
+L +12V #PWR08
 U 1 1 5123A524
 P 5050 1400
-F 0 "#PWR07" H 5050 1350 20  0001 C CNN
+F 0 "#PWR08" H 5050 1350 20  0001 C CNN
 F 1 "+12V" H 5050 1500 30  0000 C CNN
 	1    5050 1400
@@
 $EndComp
 $Comp
-L GND #PWR08
+L GND #PWR09
 U 1 1 5123A3E5
 P 6150 5650
-F 0 "#PWR08" H 6150 5650 30  0001 C CNN
+F 0 "#PWR09" H 6150 5650 30  0001 C CNN
 F 1 "GND" H 6150 5580 30  0001 C CNN
 	1    6150 5650
@@
 $EndComp
 $Comp
-L GND #PWR011
+L GND #PWR010
 U 1 1 5123A02B
 P 4100 2800
-F 0 "#PWR011" H 4100 2800 30  0001 C CNN
+F 0 "#PWR010" H 4100 2800 30  0001 C CNN
 F 1 "GND" H 4100 2730 30  0001 C CNN
 	1    4100 2800
@@
 $EndComp
 $Comp
-L +3,3V #PWR012
+L +3,3V #PWR011
 U 1 1 51239FFC
 P 7500 3100
-F 0 "#PWR012" H 7500 3060 30  0001 C CNN
+F 0 "#PWR011" H 7500 3060 30  0001 C CNN
 F 1 "+3,3V" H 7500 3210 30  0000 C CNN
 	1    7500 3100
@@
 $EndComp
 $Comp
-L GND #PWR013
+L GND #PWR012
 U 1 1 51239FFA
 P 7500 3600
-F 0 "#PWR013" H 7500 3600 30  0001 C CNN
+F 0 "#PWR012" H 7500 3600 30  0001 C CNN
 F 1 "GND" H 7500 3530 30  0001 C CNN
 	1    7500 3600
@@
 $EndComp
 $Comp
-L GND #PWR014
+L GND #PWR013
 U 1 1 51239D3F
 P 7050 5650
-F 0 "#PWR014" H 7050 5650 30  0001 C CNN
+F 0 "#PWR013" H 7050 5650 30  0001 C CNN
 F 1 "GND" H 7050 5580 30  0001 C CNN
 	1    7050 5650
@@
 $EndComp
 $Comp
-L +3,3V #PWR015
+L +3,3V #PWR014
 U 1 1 51239D16
 P 7000 4700
-F 0 "#PWR015" H 7000 4660 30  0001 C CNN
+F 0 "#PWR014" H 7000 4660 30  0001 C CNN
 F 1 "+3,3V" H 7000 4810 30  0000 C CNN
 	1    7000 4700
@@
 $EndComp
 $Comp
-L +3,3V #PWR016
+L +3,3V #PWR015
 U 1 1 5123A2F5
 P 3850 2150
-F 0 "#PWR016" H 3850 2110 30  0001 C CNN
+F 0 "#PWR015" H 3850 2110 30  0001 C CNN
 F 1 "+3,3V" H 3850 2260 30  0000 C CNN
 	1    3850 2150
@@
 $EndComp
 $Comp
-L GND #PWR017
+L GND #PWR016
 U 1 1 51239CD7
 P 7150 4750
-F 0 "#PWR017" H 7150 4750 30  0001 C CNN
+F 0 "#PWR016" H 7150 4750 30  0001 C CNN
 F 1 "GND" H 7150 4680 30  0001 C CNN
 	1    7150 4750
@@
 NoConn ~ 6500 3200
 $Comp
-L GND #PWR018
+L GND #PWR017
 U 1 1 5123A2F2
 P 4450 5100
-F 0 "#PWR018" H 4450 5100 30  0001 C CNN
+F 0 "#PWR017" H 4450 5100 30  0001 C CNN
 F 1 "GND" H 4450 5030 30  0001 C CNN
 	1    4450 5100
@@
 $EndComp
 $Comp
-L GND #PWR019
+L GND #PWR018
 U 1 1 5123A2F1
 P 3800 2600
-F 0 "#PWR019" H 3800 2600 30  0001 C CNN
+F 0 "#PWR018" H 3800 2600 30  0001 C CNN
 F 1 "GND" H 3800 2530 30  0001 C CNN
 	1    3800 2600
@@
 $EndComp
 $Comp
-L +12V #PWR020
+L +12V #PWR019
 U 1 1 5123A2EF
 P 2800 1800
-F 0 "#PWR020" H 2800 1750 20  0001 C CNN
+F 0 "#PWR019" H 2800 1750 20  0001 C CNN
 F 1 "+12V" H 2800 1900 30  0000 C CNN
 	1    2800 1800
